File: PIM_V01/PIM_V01.kicad_sch (KiCad schematic)
At the start: 13 parts, among them U1 STM32H7B3RITx, U3 TPS259814ARPWR, U5 TPS26631RGE

Commit message: ..
Parts:
- removed C10: 1uF, symbol Device:C_Small
- removed C11: 6.8nF, symbol Device:C_Small
- removed C12, C13: 2200pF, symbol Device:C_Small
- removed C15: C_Small_US, symbol Device:C_Small_US
- removed D1, D2: PTVS15VZ1USK, Diode_SMD:Nexperia_DSN1608-2_1.6x0.8mm, symbol Diode:PTVS15VZ1USK
- removed R3, R4: 4.7kR, symbol Device:R_Small
- removed R5: 1kR, symbol Device:R_Small
- removed U3: TPS259814ARPWR, VQFN10_RPW_TEX, symbol 2026-05-13_23-10-41:TPS259814ARPWR
- removed U5: TPS26631RGE, Package_DFN_QFN:Texas_RGE0024H_VQFN-24-1EP_4x4mm_P0.5mm_EP2.7x2.7mm_ThermalVias, symbol Power_Management:TPS26631RGE
- added J1: 12402143E512A, 12402143E512A:AMPHENOL_12402143E512A, symbol MyComponents:12402143E512A
- added J3: Conn_02x03_Odd_Even, symbol Connector_Generic:Conn_02x03_Odd_Even
- added U2: ~, symbol MyComponents:TPS25948x
- added U3: MCP2562-E-P, Package_DIP:DIP-8_W7.62mm, symbol Interface_CAN_LIN:MCP2562-E-P
Connections:
- net +12V_SW: now also U2.11 (VOUT), U2.6 (VOUT)
- net GND: now also J1.SH1 (SHIELD), J1.SH2 (SHIELD__1), J1.SH3 (SHIELD__2), J1.SH4 (SHIELD__3), J3.3 (Pin_3), U2.8 (GND), U3.2 (VSS)
- new net +12V_IN: U2.12 (VIN), U2.5 (VIN)
- new net +3V3: U3.3 (VDD), U3.5 (Vio)
- new net CANH: U3.7 (CANH)
- new net CANL: U3.6 (CANL)
- new net CAN_RX: U3.4 (RXD)
- new net CAN_TX: U3.1 (TXD)
- new net SWCLK: J3.2 (Pin_2)
- new net SWDIO: J3.4 (Pin_4)
- new net SWO: J3.6 (Pin_6)
- new net VREF: J3.1 (Pin_1)
- new net nRST: J3.5 (Pin_5)
Other:
- note added: "HIA INTERFACE"
- note added: "MCU"
- note added: "NEEDS TO BE FD..."
- note added: "PAYLOAD CONN"
- note added: "SWD"
- note added: "USB-C"
- note removed: "ETHERNET"
- note removed: "INPUT"
- note removed: "TPS26631 eFuse OVP, UVLO, OCP, soft-start + external B-FET"
- note removed: "need external reverse polarity fet"
- moved on the sheet: U1

Commit message: Initial commit of local KiCad project copy
Parts:
- removed U1: STM32H7B3RITx, Package_QFP:LQFP-64_10x10mm_P0.5mm, symbol MCU_ST_STM32H7:STM32H7B3RITx
- removed U3: MCP2562-E-P, Package_DIP:DIP-8_W7.62mm, symbol Interface_CAN_LIN:MCP2562-E-P
- added C1, C2, C3, C4, C5, C6, C7, C8, C9: 0.1uF, symbol Device:C_Small
- added J2, J4, J5: Screw_Terminal_01x02, symbol Connector:Screw_Terminal_01x02
- added JP1: Jumper_2_Small_Bridged, symbol Jumper:Jumper_2_Small_Bridged
- added R1, R11: 120R, symbol Device:R_Small
- added R10: 10kR, symbol Device:R_Small
- added R2, R3: xx, symbol Device:R_Small
- added R4, R5: 5k1R, symbol Device:R_Small
- added R6, R7, R8, R9: 22R, symbol Device:R_Small
- added U1, U3: MCP2562FD-H/SN, symbol MyComponents:MCP2562FD-H/SN
- added U4: STM32H7A3VITx, Package_QFP:LQFP-100_14x14mm_P0.5mm, symbol MCU_ST_STM32H7:STM32H7A3VITx
Connections:
- net +12V_IN: now also J4.1 (Pin_1), R2.1
- net +3V3: now also R10.1
- net CANH: now also J2.1 (Pin_1), J5.1 (Pin_1), R1.1, R11.1, U1.7 (CANH), U3.7 (CANH)
- net CANL: now also J2.2 (Pin_2), J5.2 (Pin_2), R1.2, R11.2, U1.6 (CANL), U3.6 (CANL)
- net CAN_RX: now also U1.4 (RXD), U3.4 (RXD)
- net CAN_TX: now also U1.1 (TXD), U3.1 (TXD)
- net GND: now also J1.A1 (GND_A), J1.A12 (GND_A__1), J1.B1 (GND_B), J1.B12 (GND_B__1), U2.1 (EN/UVLO), C1.2, C2.2, C3.2, C4.2, C5.2, J4.2 (Pin_2), R2.2, R3.1, R4.2, R5.2, U1.2 (VSS), U3.2 (VSS)
- net TX+: now reaches J1.A2 (TX1+)
- net TX+: now also J1.B3 (TX2-)
- net TX-: now reaches J1.A3 (TX1-)
- net TX-: now also J1.B2 (TX2+)
- net +5V_USB: now reaches J1.A4 (VBUS_A)
- net +5V_USB: now also J1.A9 (VBUS_A__1), J1.B4 (VBUS_B), J1.B9 (VBUS_B__1)
- net at J1.A5 (CC1): now also R4.1
- net at J1.A6 (D1+): now also R6.2
- net at J1.A7 (D1-): now also R7.2
- net at J1.B5 (CC2): now also R5.1
- net at J1.B6 (D2+): now also R9.1
- net at J1.B7 (D2-): now also R8.1
- net at U2.10 (ITIMER): now also C3.1
- net at U2.2 (OVLO): now also R3.2
- new net: U4.10 (VSS), U4.26 (VSS), U4.49 (VSS), U4.74 (VSS), U4.99 (VSS)
- new net: JP1.1 (A), U4.94 (BOOT0)
- new net: JP1.2 (B), R10.2
- new net +3V3_HKPG: C2.1, C4.1, U1.5 (VIO), U3.5 (VIO)
- new net +5V_HKPG: C1.1, C5.1, U1.3 (VDD), U3.3 (VDD)
- new net CAN_STBY: U1.8 (STBY), U3.8 (STBY)
- new net USB_D+: R6.1, R9.2
- new net USB_D-: R7.1, R8.2, U4.70 (PA11), U4.71 (PA12), U4.72 (PA13), U4.76 (PA14)
- new net USB_VBUS_SEN: U4.68 (PA9)
Other:
- sheet POWER renamed PAYLOAD_POWER
- sheet PAYLOAD_POWER ports: added +3V3_EN, +5V_EN, FAULT_IRQ, LED_STATUS, REG_EN, REG_ISENSE, REG_PGOOD, REG_SYNC, TEMP_ANA, VSEL; removed none
- note added: "SPLIT TERMINATION ON CAN"
- note added: "Will be removed for flight"
- note added: "check 22R req for D+-"
- note added: "check chat to Louis, can be flashed directly from USB!"
- note added: "need to run the stm32 AND the can transcever txrx from the same 3v3 hkpg"
- note removed: "2-pin power 12V in CAN header Satellite bus USB-C Customer sim interface, virtual COM port SWD pads Internal debug only"
- note removed: "NEEDS TO BE FD..."
- moved on the sheet: J1, J3
