File: PIM_V01/PIM_V01.kicad_sch (KiCad schematic)
At the start: 30 parts, among them J1 12402143E512A, J2 Screw_Terminal_01x02, J3 Conn_02x03_Odd_Even, J4 Screw_Terminal_01x02, J5 Screw_Terminal_01x02, U1 MCP2562FD-H/SN, U3 MCP2562FD-H/SN, U4 STM32H7A3VITx

Commit message: a month of progress, schematic is nearly done (just needs to be checked), and layout is getting close'
Parts:
- removed J1: 12402143E512A, 12402143E512A:AMPHENOL_12402143E512A, symbol MyComponents:12402143E512A
- removed J2, J4, J5: Screw_Terminal_01x02, symbol Connector:Screw_Terminal_01x02
- removed JP1: Jumper_2_Small_Bridged, symbol Jumper:Jumper_2_Small_Bridged
- removed R1: 120R, symbol Device:R_Small
- removed R9: 22R, symbol Device:R_Small
- removed U1, U3: MCP2562FD-H/SN, symbol MyComponents:MCP2562FD-H/SN
- removed U2: ~, symbol MyComponents:TPS25948x
- added C100, C64: 27pF, Capacitor_SMD:C_0603_1608Metric, symbol Device:C_Small
- added C63: 100nF, Capacitor_SMD:C_0603_1608Metric, symbol Device:C_Small
- added C78, C79, C80, C95, C99: 1uF, Capacitor_SMD:C_0603_1608Metric, symbol Device:C_Small
- added C81, C89, C90, C91, C92, C93, C98: 0.1uF, Capacitor_SMD:C_0603_1608Metric, symbol Device:C_Small
- added C82: 10uF, Capacitor_SMD:C_0603_1608Metric, symbol Device:C_Small
- added C94: 4.7uF, Capacitor_SMD:C_0603_1608Metric, symbol Device:C_Small
- added C96, C97: 2.2uF, Capacitor_SMD:C_0603_1608Metric, symbol Device:C_Small
- added D1: SMBJ13A, CustomFootprints:SMBJ16A, symbol Device:D_Zener
- added D13: SMAJ13A, Diode_SMD:D_SMA, symbol Diode:SMAJ13A
- added D2: LED, LED_SMD:LED_0603_1608Metric, symbol Device:LED
- added D3: PMEG4010, Diode_SMD:Nexperia_CFP3_SOD-123W, symbol Device:D_Schottky
- added D4: BZT52C15, Diode_SMD:Nexperia_CFP3_SOD-123W, symbol Device:D_Zener
- added J1: Conn_01x06, Connector_Molex:Molex_Pico-Lock_504050-0691_1x06-1MP_P1.50mm_Horizontal, symbol Connector_Generic:Conn_01x06
- added J10, J9: Conn_02x08_Odd_Even, Connector_PinHeader_2.54mm:PinHeader_2x08_P2.54mm_Vertical, symbol Connector_Generic:Conn_02x08_Odd_Even
- added J4: USB_C_Receptacle_USB2.0_14P, Connector_USB:USB_C_Receptacle_HCTL_HC-TYPE-C-16P-01A, symbol Connector:USB_C_Receptacle_USB2.0_14P
- added J5, J6: Conn_01x04, Connector_Molex:Molex_PicoBlade_53261-0471_1x04-1MP_P1.25mm_Horizontal, symbol Connector_Generic:Conn_01x04
- added J8: Conn_01x02, Connector_PinHeader_2.54mm:PinHeader_1x02_P2.54mm_Vertical, symbol Connector_Generic:Conn_01x02
- added Q1: SQJ407EP-T1_GE3, CustomFootprints:PowerPAK-SO-8L_Option-2_VIS, symbol Custom_Components:SQJ407EP-T1_GE3
- added Q2, Q3: PMOS, Package_TO_SOT_SMD:SOT-23-3, symbol Simulation_SPICE:PMOS
- added Q4: NMOS, Package_TO_SOT_SMD:SOT-23-3, symbol Simulation_SPICE:NMOS
- added R12, R69: 1MR, Resistor_SMD:R_0603_1608Metric, symbol Device:R_Small
- added R5: 511R, Resistor_SMD:R_0603_1608Metric, symbol Device:R_Small
- added R51, R52, R57, R58: 4.7kR, Resistor_SMD:R_0603_1608Metric, symbol Device:R_Small
- added R59, R60, R61, R66, R67: 10kR, Resistor_SMD:R_0603_1608Metric, symbol Device:R_Small
- added R62, R63, R64, R65: 33R, Resistor_SMD:R_0603_1608Metric, symbol Device:R_Small
- added R68, R70: 100kR, Resistor_SMD:R_0603_1608Metric, symbol Device:R_Small
- added SW1: SW_Push, Button_Switch_SMD:SW_SPST_B3U-1000P, symbol Switch:SW_Push
- added U1: TPS259541DSGR, CustomFootprints:DSG0008A, symbol Custom_Components:TPS259573DSGR
- added U11: AP2112K-3.3, Package_TO_SOT_SMD:SOT-23-5, symbol Regulator_Linear:AP2112K-3.3
- added U13: MT29F1G01ABAFDWB-IT_F, Package_SON:WSON-8-1EP_8x6mm_P1.27mm_EP3.4x4.3mm, symbol Custom_Components:MT29F1G01ABAFDWB-IT_F
- added U14: MB85RS256B, Package_SO:JEITA_SOIC-8_3.9x4.9mm_P1.27mm, symbol Memory_NVRAM:MB85RS256B
- added U2: USBLC6-2SC6, Package_TO_SOT_SMD:SOT-23-6, symbol Power_Protection:USBLC6-2SC6
- added Y1: Crystal_GND24_Small, Crystal:Crystal_SMD_Abracon_ABM8G-4Pin_3.2x2.5mm, symbol Device:Crystal_GND24_Small
- C1, C8: value 0.1uF -> 1uF; footprint (none) -> Capacitor_SMD:C_0603_1608Metric
- C2: footprint (none) -> Capacitor_SMD:C_0603_1608Metric
- C3: value 0.1uF -> 3.3nF; footprint (none) -> Capacitor_SMD:C_0603_1608Metric
- C4, C5: value 0.1uF -> 47uF; footprint (none) -> Capacitor_SMD:C_0603_1608Metric; Rating (none) -> 50V, MLCC
- C6, C7, C9: value 0.1uF -> 10uF; footprint (none) -> Capacitor_SMD:C_0603_1608Metric
- J7: renamed from J3; footprint (none) -> Connector_PinHeader_2.54mm:PinHeader_2x03_P2.54mm_Vertical
- R1: renamed from R4; footprint (none) -> Resistor_SMD:R_0603_1608Metric
- R11: value 120R -> 0R; footprint (none) -> Resistor_SMD:R_0603_1608Metric
- R13: renamed from R10; footprint (none) -> Resistor_SMD:R_0603_1608Metric
- R2: value xx -> 866kR; footprint (none) -> Resistor_SMD:R_0603_1608Metric
- R3: value xx -> 150kR; footprint (none) -> Resistor_SMD:R_0603_1608Metric
- R4: renamed from R5; footprint (none) -> Resistor_SMD:R_0603_1608Metric
- R6: value 22R -> 470R; footprint (none) -> Resistor_SMD:R_0603_1608Metric
- R7: value 22R -> 10kR; footprint (none) -> Resistor_SMD:R_0603_1608Metric
- R8: value 22R -> 100kR; footprint (none) -> Resistor_SMD:R_0603_1608Metric
- renumbered U4 to U3
Connections:
- net +3V3 is gone; now on net BOOT0: R13.1
- net VREF is gone; now on net +3V3_MCU: J7.1 (Pin_1)
- net +12V_IN: now also C4.1, C5.1, C6.1, D1.1 (K), J1.1 (Pin_1), J1.2 (Pin_2), J1.3 (Pin_3), Q1.5 (D); no longer R2.1
- net +3V3_EN: now also U3.97 (PE0)
- net +5V_EN: now also U3.98 (PE1)
- net +5V_USB: now also C7.1, R6.1, C78.1, C82.1, J4.A4 (VBUS), J4.A9 (VBUS), J4.B4 (VBUS), J4.B9 (VBUS), U11.1 (VIN), U11.3 (EN), U2.5 (VBUS)
- net GND: now also C3.1, C6.2, C7.2, C8.2, C9.2, J7.5 (Pin_5), R13.2, R3.2, R8.2, U3.10 (VSS), U3.19 (VSSA), U3.26 (VSS), U3.49 (VSS), U3.74 (VSS), U3.99 (VSS), C100.2, C63.2, C64.2, C78.2, C79.2, C80.2, C81.2, C82.2, C89.2, C90.2, C91.2, C92.2, C93.2, C94.2, C95.2, C96.2, C97.2, C98.2, C99.2, D1.2 (A), D13.2 (A2), D2.1 (K), D3.2 (A), J1.4 (Pin_4), J1.5 (Pin_5), J1.6 (Pin_6), J10.10 (Pin_10), J10.12 (Pin_12), J10.14 (Pin_14), J10.16 (Pin_16), J10.4 (Pin_4), J10.6 (Pin_6), J10.8 (Pin_8), J4.A1 (GND), J4.A12 (GND), J4.B1 (GND), J4.B12 (GND), J4.S1 (SHIELD), J9.10 (Pin_10), J9.12 (Pin_12), J9.14 (Pin_14), J9.2 (Pin_2), J9.4 (Pin_4), J9.6 (Pin_6), J9.8 (Pin_8), Q4.3 (S), R12.2, R5.1, R69.2, SW1.1, U1.8 (GND), U1.9 (GND), U11.2 (GND), U13.4 (VSS), U14.4 (GND), U2.2 (GND), Y1.2 (G), Y1.4 (G); no longer C3.2, R2.2, R3.1
- net SWCLK: now also J7.4 (Pin_4), U3.76 (PA14); no longer J7.2 (Pin_2)
- net SWDIO: now also J7.2 (Pin_2), U3.72 (PA13); no longer J7.4 (Pin_4)
- net SWO: now also U3.89 (PB3)
- net USB_D+: now also U3.71 (PA12), U2.6 (I/O1); no longer R6.1
- net USB_D-: now also U2.4 (I/O2); no longer R7.1, R8.2, U3.71 (PA12), U3.72 (PA13), U3.76 (PA14)
- net nRST: now also U3.14 (NRST), C63.1, SW1.2; no longer J7.5 (Pin_5)
- net +3V3_MCU: now reaches C9.1
- net +3V3_MCU: now also U3.100 (VDD), U3.11 (VDD), U3.20 (VREF+), U3.21 (VDDA), U3.27 (VDD), U3.50 (VDD), U3.6 (VBAT), U3.75 (VDD), C80.1, C81.1, C89.1, C90.1, C91.1, C92.1, C93.1, C94.1, C95.1, C98.1, C99.1, J10.2 (Pin_2), J8.2 (Pin_2), J9.1 (Pin_1), Q2.3 (S), Q3.3 (S), R51.1, R52.1, R57.2, R58.1, R59.1, R60.1, R61.1, R66.1, R67.1, R70.1, U13.8 (VCC), U14.8 (VDD)
- net at R4.1: now also J4.B5 (CC2)
- net at R1.1: now also J4.A5 (CC1)
- net at R6.2: now also D2.2 (A)
- net PL_FLT: now reaches R7.2
- net PL_FLT: now also U1.6 (FLT_N)
- net at R8.1: now also D4.2 (A), Q1.4 (G)
- net +12V_PL: now reaches C8.1
- net +12V_PL: now also D3.1 (K), U1.5 (OUT)
- net +VARI_EN: now reaches U3.1 (PE2)
- net at U3.12 (PH0): now also C100.1, Y1.1
- net at U3.13 (PH1): now also C64.1, Y1.3
- net at U3.29 (PA5): now also R62.1
- net SPI1_MISO_FPGA: now reaches U3.30 (PA6)
- net SPI1_MISO_FPGA: now also J9.7 (Pin_7)
- net at U3.31 (PA7): now also R63.1
- net OCTOSPI1_CLK: now reaches U3.36 (PB2)
- net OCTOSPI1_CLK: now also U13.6 (SCK)
- net OCTOSPI1_BK2_IO0: now reaches U3.37 (PE7)
- net OCTOSPI1_BK2_IO0: now also U13.5 (SI/IO0)
- net OCTOSPI1_BK2_IO1: now reaches U3.38 (PE8)
- net OCTOSPI1_BK2_IO1: now also U13.2 (SO/IO1)
- net OCTOSPI1_BK2_IO2: now reaches U3.39 (PE9)
- net OCTOSPI1_BK2_IO2: now also R60.2, U13.3 (WP#/IO2)
- net OCTOSPI1_BK2_IO3: now reaches U3.40 (PE10)
- net OCTOSPI1_BK2_IO3: now also R61.2, U13.7 (HOLD#/IO3)
- net SPI4_SCK_FRAM: now reaches U3.42 (PE12)
- net SPI4_SCK_FRAM: now also U14.6 (SCK)
- net SPI4_MISO_FRAM: now reaches U3.43 (PE13)
- net SPI4_MISO_FRAM: now also U14.2 (SO)
- net SPI4_MOSI_FRAM: now reaches U3.44 (PE14)
- net SPI4_MOSI_FRAM: now also U14.5 (SI)
- net SPI4_NSS_FRAM: now reaches U3.45 (PE15)
- net I2C2_SCL_PL: now reaches U3.46 (PB10)
- net I2C2_SCL_PL: now also J10.5 (Pin_5), R57.1
- net I2C2_SDA_PL: now reaches U3.47 (PB11)
- net I2C2_SDA_PL: now also J10.7 (Pin_7), R58.2
- net at U3.48 (VCAP): now also C96.1
- net CAN1_RX: now reaches U3.51 (PB12)
- net CAN1_TX: now reaches U3.52 (PB13)
- net USART3_TX_PL: now reaches U3.55 (PD8)
- net USART3_TX_PL: now also J10.1 (Pin_1)
- net USART3_RX_PL: now reaches U3.56 (PD9)
- net USART3_RX_PL: now also J10.3 (Pin_3)
- net PAYLOAD_nEN: now reaches U3.57 (PD10)
- net at U3.58 (PD11): now also R64.2
- net at U3.59 (PD12): now also R65.2
- net CDONE_FPGA: now reaches U3.60 (PD13)
- net CDONE_FPGA: now also J9.13 (Pin_13), R67.2
- net FPGA_INT: now reaches U3.61 (PD14)
- net FPGA_INT: now also J9.15 (Pin_15)
- net FPGA_EXTRA: now reaches U3.62 (PD15)
- net FPGA_EXTRA: now also J9.16 (Pin_16)
- net at U3.73 (VCAP): now also C97.1
- net OCTOSPI1_BK2_NCS: now reaches U3.79 (PC11)
- net OCTOSPI1_BK2_NCS: now also R59.2, U13.1 (CS#)
- net CAN0_RX: now reaches U3.81 (PD0)
- net CAN0_TX: now reaches U3.82 (PD1)
- net SPI2_SCK_PL: now reaches U3.84 (PD3)
- net VARI_SCL: now reaches U3.92 (PB6)
- net VARI_SCL: now also R52.2
- net VARI_SDA: now reaches U3.93 (PB7)
- net VARI_SDA: now also R51.2
- net BOOT0: now reaches U3.94 (BOOT0)
- net BOOT0: now also J8.1 (Pin_1)
- net +3V3_HKPG renamed +12V_HK
- net +12V_HK: now also C1.1, R2.1, D13.1 (A1), D4.1 (K), Q1.1 (S), Q1.2 (S), Q1.3 (S), U1.3 (IN), U1.4 (IN); no longer C4.1
- removed net +5V_HKPG: C1.1, C5.1
- net CANH: no longer names the net of R11.1
- net CANH: now also Q3.2 (G)
- net CANL renamed +3V3_HK
- net +3V3_HK: now also R7.1, Q2.1 (D), R12.1, R68.1
- new net: Q2.2 (G), Q4.1 (D), R70.2
- new net: Q4.2 (G), R68.2, R69.1
- new net: C3.2, U1.1 (DV_DT)
- new net: R2.2, R3.1, U1.2 (EN_UVLO)
- new net: R5.2, U1.7 (ILM)
- new net +3V3_USB: C79.1, Q3.1 (D), U11.5 (VOUT)
- new net CAN0_N: J5.1 (Pin_1), J5.2 (Pin_2)
- new net CAN0_P: J5.3 (Pin_3), J5.4 (Pin_4)
- new net CAN1_N: J6.1 (Pin_1), J6.2 (Pin_2)
- new net CAN1_P: J6.3 (Pin_3), J6.4 (Pin_4)
- new net D+: J4.A6 (D+), J4.B6 (D+), U2.1 (I/O1)
- new net D-: J4.A7 (D-), J4.B7 (D-), U2.3 (I/O2)
- new net SPI1_MOSI_FPGA: J9.5 (Pin_5), R63.2
- new net SPI1_SCK_FPGA: J9.3 (Pin_3), R62.2
- new net SPI4_nSS_FRAM: U14.1 (~{CS})
- new net nCRESET_FPGA: J9.11 (Pin_11), R65.1
- new net nSS_SPI_FPGA: J9.9 (Pin_9), R64.1, R66.2
Other:
- sheet PAYLOAD_POWER renamed POWER
- added sheet CAN (CAN.kicad_sch)
- sheet POWER: file POWER.kicad_sch -> PAYLOAD_POWER.kicad_sch
- sheet POWER ports: added +VARI_EN, VARI_SCL, VARI_SDA; removed FAULT_IRQ, LED_STATUS, REG_EN, REG_ISENSE, REG_PGOOD, REG_SYNC, TEMP_ANA, VSEL
- note added: "BOOT0 - selects DFU at reset"
- note added: "BOOT0 = LOW at reset → run your firmware (normal). BOOT0 = HIGH at reset → run ST's bootloader → chip shows up on the PC as a USB DFU device → we flash it."
- note added: "FPGA CONN"
- note added: "FPGA: - config: MCU as SPI master, FPGA in slave config mode - runtime:"
- note added: "INPUT POWER"
- note added: "MCU DESIGN NOTES: - MCU osc caps: load cap ≈ 2 × (CL − C_stray) = 2 × (18 − ~4.5) ≈ 27pF"
- note added: "MEMORY"
- note added: "PL CONN"
- note added: "digital OR: if USB plugged in, ability to power MCU w just +5V_USB..."
- note added: "picoblade"
- note added: "picolock"
- note added: "remove for flight 1.27 mm pitch"
- note removed: "HIA INTERFACE"
- note removed: "PAYLOAD CONN"
- note removed: "SD"
- note removed: "SPLIT TERMINATION ON CAN"
- note removed: "Will be removed for flight"
- note removed: "check chat to Louis, can be flashed directly from USB!"
- moved on the sheet: J7, R1, R13, R4, U3
