File: PIM_V01/PIM_V01.kicad_sch (KiCad schematic)
At the start: 80 parts, among them J1 Conn_01x06, J10 Conn_02x08_Odd_Even, J4 USB_C_Receptacle_USB2.0_14P, J5 Conn_01x04, J6 Conn_01x04, J7 Conn_02x03_Odd_Even, J8 Conn_01x02, J9 Conn_02x08_Odd_Even, Q1 SQJ407EP-T1_GE3, Q2 PMOS, Q3 PMOS, Q4 NMOS, SW1 SW_Push, U1 TPS259541DSGR, U11 AP2112K-3.3, U13 MT29F1G01ABAFDWB-IT_F, U14 MB85RS256B, U2 USBLC6-2SC6, U3 STM32H7A3VITx, Y1 Crystal_GND24_Small

Commit message: updated schematic to include FRAM. Ben to review soon'
Parts:
- added C103: 0.1uF, Capacitor_SMD:C_0603_1608Metric, symbol Device:C_Small
- added C104: 1uF, Capacitor_SMD:C_0603_1608Metric, symbol Device:C_Small
Connections:
- net SPI4_NSS_FRAM is gone; now on net SPI4_nSS_FRAM: U3.45 (PE15)
- net +3V3_MCU: now also U14.3 (~{WP}), U14.7 (~{HOLD}), C103.1, C104.1; no longer J10.2 (Pin_2)
- net GND: now also J10.2 (Pin_2), C103.2, C104.2
- net SPI2_SCK_PL: now also J10.9 (Pin_9)
- net SPI2_MISO_PL: now reaches U3.53 (PB14)
- net SPI2_MISO_PL: now also J10.11 (Pin_11)
- net SPI2_MOSI_PL: now reaches U3.54 (PB15)
- net SPI2_MOSI_PL: now also J10.13 (Pin_13)
- net SPI2_nCS_PL: now reaches U3.85 (PD4)
- net SPI2_nCS_PL: now also J10.15 (Pin_15)
- net PAYLOAD_nEN: no longer names the net of U3.57 (PD10)
- net USB_VBUS_SEN: no longer names the net of U3.68 (PA9)
- no-connect marks 0 -> 40

Commit message: minor updates to sch, bigger updates to pcb, after this push i am moving to double sided pcb for space optimisation
Parts:
- added D14, D15: LED, LED_SMD:LED_0603_1608Metric, symbol Device:LED
- added R79, R80: 1.8kR, Resistor_SMD:R_0603_1608Metric, symbol Device:R_Small
Connections:
- net +12V_HK: now also R79.1
- net +12V_PL: now also R80.1
- net GND: now also D14.1 (K), D15.1 (K)
- new net: D14.2 (A), R79.2
- new net: D15.2 (A), R80.2
Other:
- moved on the sheet: C4, C5, C6, D1, D4, J1, Q1, R8

Commit message: ben to review, added mounting holes and finished the rest of the layout; also labelled more of the pinouts and added leds and tps
Parts:
- added D5, D6: LED, LED_SMD:LED_0603_1608Metric, symbol Device:LED
- added H1, H2, H3, H4: MountingHole, MountingHole:MountingHole_2.2mm_M2, symbol Mechanical:MountingHole
- added R81, R82: 100R, Resistor_SMD:R_0603_1608Metric, symbol Device:R_Small
- added TP1, TP2, TP3, TP4: TestPoint, TestPoint:TestPoint_Pad_D1.0mm, symbol Connector:TestPoint
Connections:
- net CAN0_RX: now also U3.51 (PB12), TP2.1; no longer U3.81 (PD0)
- net CAN0_TX: now also U3.52 (PB13), TP1.1; no longer U3.82 (PD1)
- net CAN1_RX: now also U3.81 (PD0), TP3.1; no longer U3.51 (PB12)
- net CAN1_TX: now also U3.82 (PD1), TP4.1; no longer U3.52 (PB13)
- net GND: now also D5.1 (K), D6.1 (K)
- net TEST1_LED: now reaches U3.95 (PB8)
- net TEST1_LED: now also R81.1
- net TEST2_LED: now reaches U3.96 (PB9)
- net TEST2_LED: now also R82.1
- new net: D6.2 (A), R82.2
- new net: D5.2 (A), R81.2
- no-connect marks 40 -> 38
Other:
- note added: "BOOT0 selects DFU at reset"
- note added: "Chassis on flight"
- note added: "MOUNTING HOLES"
- note added: "R5 select on test"
- note removed: "BOOT0 - selects DFU at reset"
