File: PIM_V01/POWER.kicad_sch (KiCad schematic)
At the start: 24 parts, among them U8 TPS62933, U9 TPS62933

Commit message: Initial commit of local KiCad project copy
Connections:
- net +5V_EN: no longer U9.2 (EN)
- new net +3V3_EN: U9.2 (EN)
Other:
- moved on the sheet: C34, C35, C36, C37, C38, C39, C40, C41, C42, C43, C44, C45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
