File: PIM_V01/POWER.kicad_sch (KiCad schematic)
At the start: 114 parts, among them J11 Conn_01x02, J12 Conn_01x02, J13 Conn_01x02, U10 TPS62933, U12 MP28167GQ-A-P, U6 TPS62933, U7 TPS62933, U8 TPS62933, U9 TPS62933

Commit message: minor updates to sch, bigger updates to pcb, after this push i am moving to double sided pcb for space optimisation
Parts:
- D10, D11, D12, D9: MPN (none) -> XL-1608PGC-06; PD (none) -> CHIP LED 0603 GREEN SMD
- R32, R34: value 470R -> 100R
Changed lines of the file:
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@@
 			)
 		)
-		(property "Value" "470R"
+		(property "Value" "100R"
 			(at 151.13 237.4899 0)
 			(effects
@@
 			)
 		)
+		(property "MPN" "XL-1608PGC-06"
+			(at 148.59 243.84 90)
+			(effects
+				(font
+					(size 1.27 1.27)
+				)
+				(hide yes)
+			)
+		)
+		(property "PD" "CHIP LED 0603 GREEN SMD"
+			(at 148.59 243.84 90)
+			(effects
+				(font
+					(size 1.27 1.27)
+				)
+				(hide yes)
+			)
+		)
 		(pin "2"
 		)
@@
 			)
 		)
+		(property "MPN" "XL-1608PGC-06"
+			(at 134.62 243.84 90)
+			(effects
+				(font
+					(size 1.27 1.27)
+				)
+				(hide yes)
+			)
+		)
+		(property "PD" "CHIP LED 0603 GREEN SMD"
+			(at 134.62 243.84 90)
+			(effects
+				(font
+					(size 1.27 1.27)
+				)
+				(hide yes)
+			)
+		)
 		(pin "2"
 		)
@@
 			)
 		)
-		(property "Value" "470R"
+		(property "Value" "100R"
 			(at 185.42 237.4899 0)
 			(effects
@@
 			)
 		)
+		(property "MPN" "XL-1608PGC-06"
+			(at 182.88 243.84 90)
+			(effects
+				(font
+					(size 1.27 1.27)
+				)
+				(hide yes)
+			)
+		)
+		(property "PD" "CHIP LED 0603 GREEN SMD"
+			(at 182.88 243.84 90)
+			(effects
+				(font
+					(size 1.27 1.27)
+				)
+				(hide yes)
+			)
+		)
 		(pin "2"
 		)
@@
 			(effects
 				(font
+					(size 1.27 1.27)
+				)
+				(hide yes)
+			)
+		)
+		(property "MPN" "XL-1608PGC-06"
+			(at 168.91 243.84 90)
+			(effects
+				(font
+					(size 1.27 1.27)
+				)
+				(hide yes)
+			)
+		)
+		(property "PD" "CHIP LED 0603 GREEN SMD"
+			(at 168.91 243.84 90)
+			(effects
+				(font
