File: PIM_V01/HK_POWER.kicad_sch (KiCad schematic)
At the start: 24 parts, among them U8 TPS62933, U9 TPS62933

Commit message: a month of progress, schematic is nearly done (just needs to be checked), and layout is getting close'
Parts:
- removed C34, C35: 10uF, symbol Device:C_Small
- removed C45: 0.1uF, symbol Device:C_Small
- removed C46, C47: xxx, symbol Device:C_Small
- removed L5, L6: L_Small, symbol Device:L_Small
- removed R16, R17, R18, R19, R21: xxx, symbol Device:R_Small
- removed U8, U9: TPS62933, Package_TO_SOT_SMD:SOT-583-8, symbol Regulator_Switching:TPS62933
- added C25, C8: 0.1uF, symbol Device:C_Small
- added C6, C7: 10uF, symbol Device:C_Small
- added C9: 0.01uF, symbol Device:C_Small
- added L3, L4: L_Small, symbol Device:L_Small
- added R25, R26, R27, R28, R29: xxx, symbol Device:R_Small
- added U4, U7: TPS62933, Package_TO_SOT_SMD:SOT-583-8, symbol Regulator_Switching:TPS62933
- C36, C43: value 0.1uF -> xxx
- C37, C44: value 0.01uF -> xxx
- C38: value 0.1uF -> 10uF
- C39: value xxx -> 10uF
- C40: value xxx -> 0.1uF
- C41: value 10uF -> 0.01uF
- C42: value 10uF -> 0.1uF
Connections:
- net +12V_SW: now also C38.1, C39.1, C40.1, C6.1, C7.1, C8.1, U4.2 (EN), U4.3 (VIN), U7.2 (EN), U7.3 (VIN); no longer C36.1, C41.1, C42.1, C43.1
- net GND: now also C38.2, R20.2, C6.2, C7.2, C8.2, C9.2, R25.2, R27.2, R29.2, U4.4 (GND), U7.4 (GND); no longer C42.2
- net +5V0_HK: now reaches C37.1
- net +5V0_HK: now also C36.1, L4.2, R28.1
- net +3V3_HK: now reaches C44.1
- net +3V3_HK: now also C43.1, L3.2, R26.1
- removed net +5V: C39.1, C40.1, R20.1
- new net: R25.1, U7.1 (RT)
- new net: C25.1, U4.6 (BST)
- new net: C25.2, L4.1, U4.5 (SW)
- new net: C9.1, U4.7 (SS)
- new net: R20.1, U4.1 (RT)
- new net: R28.2, R29.1, U4.8 (FB)
- new net: C42.2, L3.1, U7.5 (SW)
- new net: C42.1, U7.6 (BST)
- new net: C41.1, U7.7 (SS)
- new net: R26.2, R27.1, U7.8 (FB)
Other:
- note removed: "+12V_SW -> +1V2"
- note removed: "+12V_SW -> +3V3"
- note removed: "+12V_SW -> +5V"
- note removed: "POWER"
- note removed: "TPS62840"
- note removed: "maybe LM61460 on the 5V rail if need 5A+"
